Commit message: update

File: aljnuho_description/urdf/aljnu_ur5e_robotiq.urdf.xacro (robot description, xacro)
@@ -3,12 +3,4 @@
     <!-- Include UR5e -->
     <xacro:include filename="$(find aljnuho_description)/urdf/ur5e/ur.urdf.xacro" />
-    <!-- Include robotiq85 adapter-->
-    <!-- <xacro:include filename="$(find aljnuho_description)/urdf/robotiq85/ur_to_robotiq_adapter.urdf.xacro" />
-    <xacro:ur_to_robotiq prefix="" connected_to="ur5e_tool0" rotation="0.0" /> -->
-    <!-- Include robotiq85 gripper -->
-    <!-- <xacro:include filename="$(find robotiq2f_description)/urdf/robotiq85/robotiq_85_macro.urdf.xacro" />
-    <xacro:robotiq_85_gripper prefix="" parent="gripper_mount_link">
-        <origin xyz="0 0 0" rpy="0 0 0" />
-    </xacro:robotiq_85_gripper> -->
     <!-- include wrist adapter -->
     <xacro:include
@@ -22,6 +14,6 @@
     </xacro:robotiq_85_gripper>
     <!-- include ros2_control -->
-    <xacro:include
+    <!-- <xacro:include
         filename="$(find robotiq2f_description)/urdf/robotiq85/robotiq_85.ros2_control.xacro" />
-    <xacro:robotiq_85_control prefix="" use_fake_hardware="$(arg use_fake_hardware)" />
+    <xacro:robotiq_85_control prefix="" use_fake_hardware="$(arg use_fake_hardware)" /> -->
 </robot>
